Commit message: decrease the camera mass from 1e-5 to 1e-8

File: models/rotors_description/urdf/component_snippets.xacro (robot description, xacro)
@@ -54,5 +54,5 @@
       </xacro:if>
       <inertial>
-        <mass value="1e-5" />
+        <mass value="1e-8" />
         <origin xyz="0 0 0" rpy="0 0 0" />
         <inertia ixx="1e-6" ixy="0" ixz="0" iyy="1e-6" iyz="0" izz="1e-6" />
